File: hardware/I2CHWC_ADCEXT/I2CHWC_ADCEXT.sch (KiCad schematic (older format))
At the start: 19 parts, among them J1 ADC 1-8, J10 EXT, J2 ADC 9-16, J3 ADC 17-24, J4 ADC 25-32, J5 ADC 33-40, J6 ADC 41-48, J7 ADC 49-56, J8 ADC 57-64, J9 ADC, U1 4051, U2 4051, U3 4051, U4 4051, U5 4051, U6 4051, U7 4051, U8 4051

Commit message: Firmwware changes: Temporarily disable ADC (whilst investigating noise issues). Change quantity of switches (from 60 to 50). Start implementing I2C commands (wip). Reverse encoder rotation (maybe just the hardware implementation of the prototype - need to validate with schematics). Schematic and PCB improvements (wip): Separate out main and extender boards to separate projects / folders. Main board now supports 10 encoders with switches, 20 switches and 8 ADC plus detection of ADC multiplex and I2C address. Extension board for encoders 11 - 30. Extension board for ADC 1 - 64.
Parts:
- removed D1: 1N4148, Diode_THT:D_DO-35_SOD27_P7.62mm_Horizontal, symbol Device:D
- added H1, H2, H3, H4: MountingHole_Pad, MountingHole:MountingHole_3.2mm_M3_Pad_Via, symbol Mechanical:MountingHole_Pad
Connections:
- wire segments 391 -> 392
Other:
- moved on the sheet: J10, J9
